Commit message: Added IMU to robot.

File: resources/simpleArm.urdf (robot description, URDF)
Before this commit: robot simpleArm, 4 links, 3 joints
Links:
- added link imu_link, mass 0.0; visual sphere radius=0.1
Joints:
- added joint imu_joint: type fixed, parent arm_3, child imu_link, origin xyz=0.0 0.0 1.0 rpy=0.0 0.0 0.0
